File: hardware/usb.kicad_sch (KiCad schematic)
At the start: 5 parts, among them J2 USB4155-03-C_REVA

Commit message: started placing leds
Parts:
- J2: footprint USB4155-03-C_REVA:GCT_USB4155-03-C_REVA -> LBD_Footprints:GCT_USB4155-03-C_REVA
Changed lines of the file:
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@@
 			)
 		)
-		(property "Footprint" "USB4155-03-C_REVA:GCT_USB4155-03-C_REVA"
+		(property "Footprint" "LBD_Footprints:GCT_USB4155-03-C_REVA"
 			(at 137.16 88.9 0)
 			(hide yes)
